File: docs/electronics/CyberwatchV1B/CyberwatchV1B.kicad_sch (KiCad schematic)
At the start: 15 parts, among them J1 Micro_SD_Card, J2 Conn_01x08, SW1 SW_Push, SW2 SW_Push, SW3 SW_Push, SW4 SW_Push, SW5 SW_SPDT, U1 XIAO-ESP32-S3-Plus-SMD, U2 MCP23017x-x-ML, U3 DS3231MZ, U4 AS5600

Commit message: electronics+case
Parts:
- removed C1: C_Small, symbol Device:C_Small
- removed J2: Conn_01x08, Connector_JST:JST_GH_SM09B-GHS-TB_1x09-1MP_P1.25mm_Horizontal, symbol Connector_Generic:Conn_01x08
- removed SW5: SW_SPDT, symbol Switch:SW_SPDT
- added BT1: Battery_Cell, symbol Device:Battery_Cell
- added C3, C4: C_Small, symbol Device:C_Small
- added J2: Conn_01x08_Display, symbol CY_library:Conn_01x08
- added Q1: AO3401A, Package_TO_SOT_SMD:SOT-23, symbol Transistor_FET:AO3401A
- added SW6: SW_power, symbol Switch:SW_SPST
Connections:
- net +3.3V: now reaches U3.2 (VCC)
- net +3.3V: now also C2.2, J1.4 (VDD), J2.1 (VCC)
- net GND: now reaches U3.5 (GND)
- net GND: now also J1.6 (VSS), U1.33 (GND), U4.4 (GND), U4.5 (DIR), J2.2 (GND)
- net at U3.6 (VBAT): now also BT1.1 (+)
- net I2C_SDA: now reaches R1.1
- net I2C_SDA: now also U1.5 (D4), U2.9 (SDA)
- net at U2.17 (GPA0): now also J2.7 (Pin_7)
- net at U2.18 (GPA1): now also J2.8 (Pin_8)
- net at U2.19 (GPA2): now also SW4.2
- net at U2.20 (GPA3): now also SW3.2
- net at U2.21 (GPA4): now also SW2.2
- net at U2.22 (GPA5): now also SW1.2
- net I2C_SCL: now reaches U2.8 (SCL)
- net I2C_SCL: now also R2.1, U1.6 (D5)
- net at U1.10 (D9): now also J1.2 (DAT3/CD)
- net SPI_MOSI: now reaches U1.11 (D10)
- net SPI_MOSI: now also J1.3 (CMD), J2.3 (DIN)
- net at U1.2 (D1): now also J2.5 (CS)
- net at U1.4 (D3): now also J2.6 (Pin_6)
- net at U1.8 (D7): now also J1.7 (DAT0)
- net SPI_CLK: now reaches U1.9 (D8)
- net SPI_CLK: now also J1.5 (CLK), J2.4 (Pin_4)
- no-connect marks 0 -> 15
Other:
- moved on the sheet: C2, J1, R1, R2, SW1, SW2, SW3, SW4, U1, U2, U3, U4
