File: design/electronics2/CyberwatchV1B/power.kicad_sch (KiCad schematic)
At the start: 4 parts, among them Q1 AO3401A, SW6 SW_power

Commit message: power schematic progres
Parts:
- removed C3, C4: C_Small, symbol Device:C_Small
- added J3: Conn_01x02_Socket, Connector_JST:JST_PH_S2B-PH-SM4-TB_1x02-1MP_P2.00mm_Horizontal, symbol Connector:Conn_01x02_Socket
- added R1: 33, symbol Device:R
- added R2: 100k, symbol Device:R
- added U4: MAX17048, symbol CY_library:MAX17048
Connections:
- net at Q1.1 (G): now also R1.1, R2.2
- net VBAT_RAW: now reaches Q1.2 (S)
- net VBAT_RAW: now also J3.1 (Pin_1), R1.2
- net VBAT_SWITCHED: now reaches Q1.3 (D)
- net at SW6.1 (A): now also R2.1
- net GND: now reaches SW6.2 (B)
- net GND: now also J3.2 (Pin_2)
- new net SCL: U4. (QSTRT)
- new net SDA: U4. (QSTRT)
Other:
- note added: "G"
- moved on the sheet: Q1, SW6

Commit message: power update confirm
Connections:
- net GND: now also U4. (QSTRT)
- net VBAT_RAW: no longer R1.2
- net VBAT_SWITCHED: now also U4.1 (VDD)
- net at Q1.1 (G), R2.2: now also R1.2; no longer R1.1
- new net ALRT: U4. (QSTRT)
Other:
- moved on the sheet: J3, Q1, R1, U4

Commit message: power schematic finalisation
Connections:
- net VBAT_RAW: now also R1.1
Other:
- moved on the sheet: J3, Q1, R1, R2, SW6, U4

Commit message: electronics progres
Parts:
- added J9: Conn_01x07_main, symbol Connector_Generic:Conn_01x07
- R1, R2: footprint (none) -> Resistor_SMD:R_0603_1608Metric
Connections:
- net ALRT: now also U4.5 (ALRT); no longer U4. (QSTRT)
- net GND: now also U4.3 (CTG), U4.4 (GND), U4.8 (QSTRT), J9.3 (Pin_3); no longer U4. (QSTRT)
- net SCL: now also U4.7 (SCL); no longer U4. (QSTRT)
- net SDA: now also U4.6 (SDA); no longer U4. (QSTRT)
- net VBAT_RAW: now also J9.1 (Pin_1)
- net VBAT_SWITCHED: now also J9.2 (Pin_2)
- net G: now reaches Q1.1 (G), R1.2, R2.2
Other:
- note removed: "G"

Commit message: schematic complete
Connections:
- net ALRT is gone; now on net PWR_ALRT: U4.5 (ALRT)
- net GND: now also J9.7 (Pin_7)
- net SCL: now also J9.5 (Pin_5)
- net SDA: now also J9.4 (Pin_4)
- net PWR_ALRT: now reaches J9.6 (Pin_6)
Other:
- moved on the sheet: J9

Commit message: sync
Parts:
- J9: value Conn_01x07_main -> Conn_01x07_PWR_main; footprint (none) -> Connector_JST:JST_SH_SM07B-SRSS-TB_1x07-1MP_P1.00mm_Horizontal
- SW6: footprint (none) -> Button_Switch_SMD:SW_DIP_SPSTx01_Slide_Copal_CHS-01A_W5.08mm_P1.27mm_JPin
- U4: footprint (none) -> Package_DFN_QFN:TDFN-8-1EP_2x2mm_P0.5mm_EP0.8x1.2mm
Changed lines of the file:
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@@
 			)
 		)
-		(property "Footprint" ""
+		(property "Footprint" "Package_DFN_QFN:TDFN-8-1EP_2x2mm_P0.5mm_EP0.8x1.2mm"
 			(at 151.13 87.63 0)
-			(hide yes)
 			(show_name no)
 			(do_not_autoplace no)
@@
 			)
 		)
-		(property "Value" "Conn_01x07_main"
+		(property "Value" "Conn_01x07_PWR_main"
 			(at 205.486 62.23 0)
 			(show_name no)
@@
 			)
 		)
-		(property "Footprint" ""
+		(property "Footprint" "Connector_JST:JST_SH_SM07B-SRSS-TB_1x07-1MP_P1.00mm_Horizontal"
 			(at 217.17 73.66 0)
 			(hide yes)
@@
 			)
 		)
-		(property "Footprint" ""
+		(property "Footprint" "Button_Switch_SMD:SW_DIP_SPSTx01_Slide_Copal_CHS-01A_W5.08mm_P1.27mm_JPin"
 			(at 149.86 120.65 0)
 			(hide yes)
