File: design/electronics2/CyberwatchV1B/CyberwatchV1B.kicad_sch (KiCad schematic)
At the start: 4 parts, among them SW1 SW_Push, SW2 SW_Push, SW3 SW_Push, SW4 SW_Push

Commit message: power schematic progres
Parts:
- removed SW1, SW2, SW3, SW4: SW_Push, symbol Switch:SW_Push
Other:
- removed sheet crown
- added sheet input_left (input_left.kicad_sch)
- added sheet input_right (input_right.kicad_sch)

Commit message: power schematic finalisation
Other:
- sheet main ports: added VBAT_RAW, VBAT_SWITCHED; removed none
- sheet power ports: added ALRT, GND, SCL, SDA, VBAT_RAW, VBAT_SWITCHED; removed none
Changed lines of the file:
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@@
 		(company "Edward Swingler")
+	)
+	(wire
+		(pts
+			(xy 124.46 67.31) (xy 124.46 76.2)
+		)
+		(stroke
+			(width 0)
+			(type default)
+		)
+	)
+	(wire
+		(pts
+			(xy 134.62 67.31) (xy 134.62 76.2)
+		)
+		(stroke
+			(width 0)
+			(type default)
+		)
 	)
 	(sheet
@@
 			)
 		)
+		(pin "VBAT_RAW" input
+			(at 134.62 76.2 90)
+			(effects
+				(font
+					(size 1.27 1.27)
+				)
+				(justify right)
+			)
+		)
+		(pin "VBAT_SWITCHED" input
+			(at 124.46 76.2 90)
+			(effects
+				(font
+					(size 1.27 1.27)
+				)
+				(justify right)
+			)
+		)
 		(instances
 			(project "CyberwatchV1B"
@@
 	)
 	(sheet
-		(at 25.4 24.13)
-		(size 254 39.37)
+		(at 120.65 44.45)
+		(size 55.88 22.86)
 		(exclude_from_sim no)
 		(in_bom yes)
@@
 		)
 		(property "Sheetname" "power"
-			(at 25.4 23.4184 0)
+			(at 119.9384 67.31 90)
 			(show_name no)
 			(do_not_autoplace no)
@@
 		)
 		(property "Sheetfile" "power.kicad_sch"
-			(at 25.4 64.0846 0)
+			(at 177.1146 67.31 90)
 			(show_name no)
 			(do_not_autoplace no)
@@
 			)
 		)
+		(pin "ALRT" output
+			(at 172.72 67.31 270)
+			(effects
+				(font
+					(size 1.27 1.27)
+				)
+				(justify left)
+			)
+		)
+		(pin "GND" output
+			(at 163.83 67.31 270)
+			(effects
+				(font
+					(size 1.27 1.27)
+				)
+				(justify left)
+			)
+		)
+		(pin "SCL" input
+			(at 153.67 67.31 270)
+			(effects
+				(font
+					(size 1.27 1.27)
+				)
+				(justify left)
+			)
+		)
+		(pin "SDA" bidirectional
+			(at 143.51 67.31 270)
+			(effects
+				(font
+					(size 1.27 1.27)
+				)
+				(justify left)
+			)
+		)
+		(pin "VBAT_RAW" output
+			(at 134.62 67.31 270)
+			(effects
+				(font
+					(size 1.27 1.27)
+				)
+				(justify left)
+			)
+		)
+		(pin "VBAT_SWITCHED" output
+			(at 124.46 67.31 270)
+			(effects
+				(font
+					(size 1.27 1.27)
+				)
+				(justify left)
+			)
+		)

Commit message: documentation and electronics main board progress
Other:
- sheet main ports: added BTN_1, BTN_2, GND, SCL, SDA; removed none
Changed lines of the file:
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@@
 	(wire
 		(pts
-			(xy 124.46 67.31) (xy 124.46 76.2)
-		)
-		(stroke
-			(width 0)
-			(type default)
-		)
-	)
-	(wire
-		(pts
-			(xy 134.62 67.31) (xy 134.62 76.2)
+			(xy 127 67.31) (xy 127 76.2)
+		)
+		(stroke
+			(width 0)
+			(type default)
+		)
+	)
+	(wire
+		(pts
+			(xy 114.3 67.31) (xy 114.3 76.2)
+		)
+		(stroke
+			(width 0)
+			(type default)
+		)
+	)
+	(wire
+		(pts
+			(xy 177.8 67.31) (xy 177.8 76.2)
+		)
+		(stroke
+			(width 0)
+			(type default)
+		)
+	)
+	(wire
+		(pts
+			(xy 165.1 67.31) (xy 165.1 76.2)
+		)
+		(stroke
+			(width 0)
+			(type default)
+		)
+	)
+	(wire
+		(pts
+			(xy 152.4 67.31) (xy 152.4 76.2)
 		)
 		(stroke
@@
 		)
 		(pin "VBAT_RAW" input
-			(at 134.62 76.2 90)
+			(at 114.3 76.2 90)
 			(effects
 				(font
@@
 		)
 		(pin "VBAT_SWITCHED" input
-			(at 124.46 76.2 90)
+			(at 127 76.2 90)
+			(effects
+				(font
+					(size 1.27 1.27)
+				)
+				(justify right)
+			)
+		)
+		(pin "BTN_1" input
+			(at 101.6 102.87 180)
+			(effects
+				(font
+					(size 1.27 1.27)
+				)
+				(justify left)
+			)
+		)
+		(pin "BTN_2" input
+			(at 101.6 105.41 180)
+			(effects
+				(font
+					(size 1.27 1.27)
+				)
+				(justify left)
+			)
+		)
+		(pin "GND" input
+			(at 177.8 76.2 90)
+			(effects
+				(font
+					(size 1.27 1.27)
+				)
+				(justify right)
+			)
+		)
+		(pin "SCL" input
+			(at 165.1 76.2 90)
+			(effects
+				(font
+					(size 1.27 1.27)
+				)
+				(justify right)
+			)
+		)
+		(pin "SDA" input
+			(at 152.4 76.2 90)
 			(effects
 				(font
@@
 	)
 	(sheet
-		(at 120.65 44.45)
-		(size 55.88 22.86)
+		(at 101.6 44.45)
+		(size 101.6 22.86)
 		(exclude_from_sim no)
 		(in_bom yes)
@@
 		)
 		(property "Sheetname" "power"
-			(at 119.9384 67.31 90)
+			(at 100.8884 67.31 90)
 			(show_name no)
 			(do_not_autoplace no)
@@
 		)
 		(property "Sheetfile" "power.kicad_sch"
-			(at 177.1146 67.31 90)
+			(at 203.7846 67.31 90)
 			(show_name no)
 			(do_not_autoplace no)
@@
 		)
 		(pin "ALRT" output
-			(at 172.72 67.31 270)
+			(at 139.7 67.31 270)
 			(effects
 				(font
@@
 		)
 		(pin "GND" output
-			(at 163.83 67.31 270)
+			(at 177.8 67.31 270)
 			(effects
 				(font
@@
 		)
 		(pin "SCL" input
-			(at 153.67 67.31 270)
+			(at 165.1 67.31 270)
 			(effects
 				(font
@@
 		)
 		(pin "SDA" bidirectional
-			(at 143.51 67.31 270)
+			(at 152.4 67.31 270)
 			(effects
 				(font
@@
 		)
 		(pin "VBAT_RAW" output
-			(at 134.62 67.31 270)
+			(at 114.3 67.31 270)
 			(effects
 				(font
@@
 		)
 		(pin "VBAT_SWITCHED" output
-			(at 124.46 67.31 270)
-			(effects
-				(font
+			(at 127 67.31 270)
+			(effects
+				(font

Commit message: electronics progres
Other:
- sheet input_left ports: added BTN_1, BTN_2; removed none
- sheet input_right ports: added BTN_3, BTN_4, SCL, SDA; removed none
- sheet main ports: added ALRT, BTN_3, BTN_4; removed GND
- sheet power ports: added none; removed GND
Changed lines of the file:
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@@
 	(wire
 		(pts
-			(xy 127 67.31) (xy 127 76.2)
-		)
-		(stroke
-			(width 0)
-			(type default)
-		)
-	)
-	(wire
-		(pts
-			(xy 114.3 67.31) (xy 114.3 76.2)
-		)
-		(stroke
-			(width 0)
-			(type default)
-		)
-	)
-	(wire
-		(pts
-			(xy 177.8 67.31) (xy 177.8 76.2)
-		)
-		(stroke
-			(width 0)
-			(type default)
-		)
-	)
-	(wire
-		(pts
-			(xy 165.1 67.31) (xy 165.1 76.2)
-		)
-		(stroke
-			(width 0)
-			(type default)
-		)
-	)
-	(wire
-		(pts
-			(xy 152.4 67.31) (xy 152.4 76.2)
-		)
-		(stroke
-			(width 0)
-			(type default)
+			(xy 214.63 127) (xy 215.9 127)
+		)
+		(stroke
+			(width 0)
+			(type default)
+		)
+	)
+	(wire
+		(pts
+			(xy 203.2 101.6) (xy 215.9 101.6)
+		)
+		(stroke
+			(width 0)
+			(type default)
+		)
+	)
+	(wire
+		(pts
+			(xy 88.9 114.3) (xy 101.6 114.3)
+		)
+		(stroke
+			(width 0)
+			(type default)
+		)
+	)
+	(wire
+		(pts
+			(xy 127 60.96) (xy 127 76.2)
+		)
+		(stroke
+			(width 0)
+			(type default)
+		)
+	)
+	(wire
+		(pts
+			(xy 214.63 139.7) (xy 215.9 139.7)
+		)
+		(stroke
+			(width 0)
+			(type default)
+		)
+	)
+	(wire
+		(pts
+			(xy 203.2 114.3) (xy 215.9 114.3)
+		)
+		(stroke
+			(width 0)
+			(type default)
+		)
+	)
+	(wire
+		(pts
+			(xy 114.3 60.96) (xy 114.3 76.2)
+		)
+		(stroke
+			(width 0)
+			(type default)
+		)
+	)
+	(wire
+		(pts
+			(xy 152.4 62.23) (xy 152.4 60.96)
+		)
+		(stroke
+			(width 0)
+			(type default)
+		)
+	)
+	(wire
+		(pts
+			(xy 88.9 101.6) (xy 101.6 101.6)
+		)
+		(stroke
+			(width 0)
+			(type default)
+		)
+	)
+	(wire
+		(pts
+			(xy 139.7 60.96) (xy 139.7 76.2)
+		)
+		(stroke
+			(width 0)
+			(type default)
+		)
+	)
+	(wire
+		(pts
+			(xy 165.1 62.23) (xy 165.1 60.96)
+		)
+		(stroke
+			(width 0)
+			(type default)
+		)
+	)
+	(wire
+		(pts
+			(xy 152.4 74.93) (xy 152.4 76.2)
+		)
+		(stroke
+			(width 0)
+			(type default)
+		)
+	)
+	(wire
+		(pts
+			(xy 165.1 74.93) (xy 165.1 76.2)
+		)
+		(stroke
+			(width 0)
+			(type default)
+		)
+	)
+	(label "SDA"
+		(at 214.63 127 180)
+		(effects
+			(font
+				(size 1.27 1.27)
+			)
+			(justify right bottom)
+		)
+	)
+	(label "SCL"
+		(at 165.1 74.93 90)
+		(effects
+			(font
+				(size 1.27 1.27)
+			)
+			(justify left bottom)
+		)
+	)
+	(label "SCL"
+		(at 214.63 139.7 180)
+		(effects
+			(font
+				(size 1.27 1.27)
+			)
+			(justify right bottom)
+		)
+	)
+	(label "SDA"
+		(at 152.4 62.23 270)
+		(effects
+			(font
+				(size 1.27 1.27)
+			)
+			(justify right bottom)
+		)
+	)
+	(label "SCL"
+		(at 165.1 62.23 270)
+		(effects
+			(font
+				(size 1.27 1.27)
+			)
+			(justify right bottom)
+		)
+	)
+	(label "SDA"
+		(at 152.4 74.93 90)
+		(effects
+			(font
+				(size 1.27 1.27)
+			)
+			(justify left bottom)
 		)
 	)
@@
 			)
 		)
+		(pin "BTN_3" input
+			(at 215.9 101.6 180)
+			(effects
+				(font
+					(size 1.27 1.27)
+				)
+				(justify left)
+			)
+		)
+		(pin "BTN_4" input
+			(at 215.9 114.3 180)
+			(effects
+				(font
+					(size 1.27 1.27)
+				)
+				(justify left)
+			)
+		)
+		(pin "SCL" input
+			(at 215.9 139.7 180)
+			(effects
+				(font
+					(size 1.27 1.27)
+				)
+				(justify left)
+			)
+		)
+		(pin "SDA" input
+			(at 215.9 127 180)
+			(effects
+				(font
+					(size 1.27 1.27)
+				)
+				(justify left)
+			)
+		)
 		(instances
 			(project "CyberwatchV1B"
@@
 		)
 		(pin "BTN_1" input
-			(at 101.6 102.87 180)
+			(at 101.6 101.6 180)
 			(effects
 				(font
@@
 		)
 		(pin "BTN_2" input
-			(at 101.6 105.41 180)
-			(effects
-				(font
-					(size 1.27 1.27)
-				)
-				(justify left)
-			)
-		)
-		(pin "GND" input
-			(at 177.8 76.2 90)
-			(effects
-				(font
-					(size 1.27 1.27)
-				)
-				(justify right)
+			(at 101.6 114.3 180)
+			(effects
+				(font
+					(size 1.27 1.27)
+				)
+				(justify left)
 			)
 		)
@@
 		(pin "SDA" input
 			(at 152.4 76.2 90)
+			(effects
+				(font
+					(size 1.27 1.27)
+				)
+				(justify right)
+			)
+		)
+		(pin "ALRT" input
+			(at 139.7 76.2 90)
+			(effects
+				(font
+					(size 1.27 1.27)
+				)
+				(justify right)
+			)
+		)
+		(pin "BTN_3" input
+			(at 203.2 101.6 0)
+			(effects
+				(font
+					(size 1.27 1.27)
+				)
+				(justify right)
+			)
+		)
+		(pin "BTN_4" input
+			(at 203.2 114.3 0)
 			(effects
 				(font
@@
 	)
 	(sheet
-		(at 101.6 44.45)
+		(at 101.6 38.1)
 		(size 101.6 22.86)
 		(exclude_from_sim no)
@@
 		)
 		(property "Sheetname" "power"
-			(at 100.8884 67.31 90)
+			(at 100.8884 60.96 90)
 			(show_name no)
 			(do_not_autoplace no)
@@
 		)
 		(property "Sheetfile" "power.kicad_sch"
-			(at 203.7846 67.31 90)
+			(at 203.7846 60.96 90)
 			(show_name no)
 			(do_not_autoplace no)
@@
 		)
 		(pin "ALRT" output
-			(at 139.7 67.31 270)
-			(effects
-				(font
-					(size 1.27 1.27)
-				)
-				(justify left)
-			)
-		)
-		(pin "GND" output
-			(at 177.8 67.31 270)
+			(at 139.7 60.96 270)
 			(effects
 				(font
@@
 		)
 		(pin "SCL" input
-			(at 165.1 67.31 270)
+			(at 165.1 60.96 270)
 			(effects
 				(font
@@
 		)
 		(pin "SDA" bidirectional
-			(at 152.4 67.31 270)
+			(at 152.4 60.96 270)
 			(effects
 				(font
@@
 		)
 		(pin "VBAT_RAW" output
-			(at 114.3 67.31 270)
+			(at 114.3 60.96 270)
 			(effects
 				(font
@@
 		)
 		(pin "VBAT_SWITCHED" output
-			(at 127 67.31 270)
+			(at 127 60.96 270)
 			(effects
 				(font
@@
 			)
 		)
+		(pin "BTN_1" input
+			(at 88.9 101.6 0)
+			(effects
+				(font
+					(size 1.27 1.27)
+				)
+				(justify right)
+			)
+		)
+		(pin "BTN_2" input
+			(at 88.9 114.3 0)
+			(effects
+				(font
+					(size 1.27 1.27)
+				)
+				(justify right)
+			)
+		)

Commit message: schematic complete
Other:
- sheet main ports: added PWR_ALRT; removed ALRT
- sheet power ports: added PWR_ALRT; removed ALRT
Changed lines of the file:
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@@
 			)
 		)
-		(pin "ALRT" input
+		(pin "PWR_ALRT" input
 			(at 139.7 76.2 90)
 			(effects
@@
 			)
 		)
-		(pin "ALRT" output
+		(pin "PWR_ALRT" output
 			(at 139.7 60.96 270)
 			(effects

Commit message: pcb design
Other:
- removed sheet power
- sheet main ports: added none; removed PWR_ALRT, VBAT_RAW, VBAT_SWITCHED
