File: design/electronics2/CyberwatchV1B/input_left.kicad_sch (KiCad schematic)
At the start: 0 parts

Commit message: electronics progres
Parts:
- added J7: Conn_01x03_main, symbol Connector_Generic:Conn_01x03
- added SW1, SW2: SW_Push, Button_Switch_SMD:SW_Push_1P1T_NO_CK_KMR2, symbol Switch:SW_Push
Connections:
- new net BTN_1: SW1.2
- new net BTN_2: SW2.2
- new net GND: SW1.1, SW2.1

Commit message: schematic complete
Connections:
- net BTN_1: now also J7.2 (Pin_2)
- net BTN_2: now also J7.3 (Pin_3)
- net GND: now also J7.1 (Pin_1)
Changed lines of the file:
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@@
 	(generator_version "10.0")
 	(paper "A4")
-	(wire
-		(pts
-			(xy 168.91 104.14) (xy 171.45 104.14)
+	(junction
+		(at 190.5 99.06)
+		(diameter 0)
+		(color 0 0 0 0)
+	)
+	(junction
+		(at 190.5 101.6)
+		(diameter 0)
+		(color 0 0 0 0)
+	)
+	(wire
+		(pts
+			(xy 186.69 104.14) (xy 186.69 101.6)
+		)
+		(stroke
+			(width 0)
+			(type default)
+		)
+	)
+	(wire
+		(pts
+			(xy 186.69 99.06) (xy 186.69 93.98)
+		)
+		(stroke
+			(width 0)
+			(type default)
+		)
+	)
+	(wire
+		(pts
+			(xy 168.91 104.14) (xy 186.69 104.14)
 		)
 		(stroke
@@
 	(wire
 		(pts
-			(xy 168.91 93.98) (xy 171.45 93.98)
+			(xy 186.69 101.6) (xy 190.5 101.6)
+		)
+		(stroke
+			(width 0)
+			(type default)
+		)
+	)
+	(wire
+		(pts
+			(xy 198.12 101.6) (xy 190.5 101.6)
+		)
+		(stroke
+			(width 0)
+			(type default)
+		)
+	)
+	(wire
+		(pts
+			(xy 198.12 96.52) (xy 190.5 96.52)
+		)
+		(stroke
+			(width 0)
+			(type default)
+		)
+	)
+	(wire
+		(pts
+			(xy 168.91 93.98) (xy 186.69 93.98)
+		)
+		(stroke
+			(width 0)
+			(type default)
+		)
+	)
+	(wire
+		(pts
+			(xy 186.69 99.06) (xy 190.5 99.06)
+		)
+		(stroke
+			(width 0)
+			(type default)
+		)
+	)
+	(wire
+		(pts
+			(xy 198.12 99.06) (xy 190.5 99.06)
 		)
 		(stroke
@@
 	(hierarchical_label "BTN_1"
 		(shape input)
-		(at 171.45 93.98 0)
+		(at 198.12 99.06 0)
 		(effects
 			(font
@@
 	(hierarchical_label "BTN_2"
 		(shape input)
-		(at 171.45 104.14 0)
+		(at 198.12 101.6 0)
 		(effects
 			(font
@@
 	)
 	(symbol
+		(lib_id "Connector_Generic:Conn_01x03")
+		(at 195.58 99.06 0)
+		(unit 1)
+		(body_style 1)
+		(exclude_from_sim no)
+		(in_bom yes)
+		(on_board yes)
+		(in_pos_files yes)
+		(dnp no)
+		(property "Reference" "J7"
+			(at 197.612 93.218 0)
+			(show_name no)
+			(do_not_autoplace no)
+			(effects
+				(font
+					(size 1.27 1.27)
+				)
+			)
+		)
+		(property "Value" "Conn_01x03_main"
+			(at 197.612 90.678 0)
+			(show_name no)
+			(do_not_autoplace no)
+			(effects
+				(font
+					(size 1.27 1.27)
+				)
+			)
+		)
+		(property "Footprint" ""
+			(at 195.58 99.06 0)
+			(hide yes)
+			(show_name no)
+			(do_not_autoplace no)
+			(effects
+				(font
+					(size 1.27 1.27)
+				)
+			)
+		)
+		(property "Datasheet" ""
+			(at 195.58 99.06 0)
+			(hide yes)
+			(show_name no)
+			(do_not_autoplace no)
+			(effects
+				(font
+					(size 1.27 1.27)
+				)
+			)
+		)
+		(property "Description" "Generic connector, single row, 01x03, script generated (kicad-library-utils/schlib/autogen/connector/)"
+			(at 195.58 99.06 0)
+			(hide yes)
+			(show_name no)
+			(do_not_autoplace no)
+			(effects
+				(font
+					(size 1.27 1.27)
+				)
+			)
+		)
+		(pin "1"
+		)
+		(pin "3"
+		)
+		(pin "2"
+		)
+		(instances
+			(project "CyberwatchV1B"
+				(path "/68fdecbc-307b-4175-ba1b-687d291eebec/ea0244fb-2f59-483a-a25c-2656c752d645"
+					(reference "J7")
+					(unit 1)
+				)
+			)
+		)
+	)
+	(symbol
 		(lib_id "Switch:SW_Push")
 		(at 163.83 93.98 0)
@@
 	)
 	(symbol
-		(lib_id "Connector_Generic:Conn_01x03")
-		(at 95.25 95.25 180)
+		(lib_id "power:GND")
+		(at 198.12 96.52 90)
+		(mirror x)
 		(unit 1)
 		(body_style 1)
@@
 		(in_pos_files yes)
 		(dnp no)
-		(fields_autoplaced yes)
-		(property "Reference" "J7"
-			(at 95.25 86.36 0)
-			(show_name no)
-			(do_not_autoplace no)
-			(effects
-				(font
-					(size 1.27 1.27)
-				)
-			)
-		)
-		(property "Value" "Conn_01x03_main"
-			(at 95.25 88.9 0)
+		(property "Reference" "#PWR044"
+			(at 204.47 96.52 0)
+			(hide yes)
+			(show_name no)
+			(do_not_autoplace no)
+			(effects
+				(font
+					(size 1.27 1.27)
+				)
+			)
+		)
+		(property "Value" "GND"
+			(at 203.454 96.52 90)
 			(show_name no)
 			(do_not_autoplace no)
@@
 		)
 		(property "Footprint" ""
-			(at 95.25 95.25 0)
+			(at 198.12 96.52 0)
 			(hide yes)
 			(show_name no)
@@
 		)
 		(property "Datasheet" ""
-			(at 95.25 95.25 0)
-			(hide yes)
-			(show_name no)
-			(do_not_autoplace no)
-			(effects
-				(font
-					(size 1.27 1.27)
-				)
-			)
-		)
-		(property "Description" "Generic connector, single row, 01x03, script generated (kicad-library-utils/schlib/autogen/connector/)"
-			(at 95.25 95.25 0)
+			(at 198.12 96.52 0)
+			(hide yes)
+			(show_name no)
+			(do_not_autoplace no)
+			(effects
+				(font
+					(size 1.27 1.27)
+				)
+			)
+		)
+		(property "Description" "Power symbol creates a global label with name \"GND\" , ground"
+			(at 198.12 96.52 0)
 			(hide yes)
 			(show_name no)
@@
 		)
 		(pin "1"
-		)
-		(pin "3"
-		)
-		(pin "2"
 		)
 		(instances
 			(project "CyberwatchV1B"
 				(path "/68fdecbc-307b-4175-ba1b-687d291eebec/ea0244fb-2f59-483a-a25c-2656c752d645"
-					(reference "J7")
+					(reference "#PWR044")
 					(unit 1)
 				)

Commit message: sync
Parts:
- J7: value Conn_01x03_main -> Conn_01x03_IL_main; footprint (none) -> Connector_JST:JST_SH_SM03B-SRSS-TB_1x03-1MP_P1.00mm_Horizontal
Changed lines of the file:
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@@
 			)
 		)
-		(property "Value" "Conn_01x03_main"
+		(property "Value" "Conn_01x03_IL_main"
 			(at 197.612 90.678 0)
 			(show_name no)
@@
 			)
 		)
-		(property "Footprint" ""
+		(property "Footprint" "Connector_JST:JST_SH_SM03B-SRSS-TB_1x03-1MP_P1.00mm_Horizontal"
 			(at 195.58 99.06 0)
 			(hide yes)

Commit message: pcb design
Parts:
- J6: renamed from J7; KiLib_Generator (none) -> connector/SMD_single_row_plus_mounting_pad
- renumbered SW1 to SW2, SW2 to SW3
Changed lines of the file:
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@@
 		(dnp no)
 		(fields_autoplaced yes)
-		(property "Reference" "#PWR023"
+		(property "Reference" "#PWR030"
 			(at 149.86 104.14 0)
 			(hide yes)
@@
 			(project "CyberwatchV1B"
 				(path "/68fdecbc-307b-4175-ba1b-687d291eebec/ea0244fb-2f59-483a-a25c-2656c752d645"
-					(reference "#PWR023")
+					(reference "#PWR030")
 					(unit 1)
 				)
@@
 		(in_pos_files yes)
 		(dnp no)
-		(property "Reference" "J7"
+		(property "Reference" "J6"
 			(at 197.612 93.218 0)
 			(show_name no)
@@
 			)
 		)
+		(property "KiLib_Generator" "connector/SMD_single_row_plus_mounting_pad"
+			(at 195.58 99.06 0)
+			(hide yes)
+			(show_name no)
+			(do_not_autoplace no)
+			(effects
+				(font
+					(size 1.27 1.27)
+				)
+			)
+		)
 		(pin "1"
 		)
@@
 			(project "CyberwatchV1B"
 				(path "/68fdecbc-307b-4175-ba1b-687d291eebec/ea0244fb-2f59-483a-a25c-2656c752d645"
-					(reference "J7")
+					(reference "J6")
 					(unit 1)
 				)
@@
 		(dnp no)
 		(fields_autoplaced yes)
-		(property "Reference" "SW1"
+		(property "Reference" "SW2"
 			(at 163.83 86.36 0)
 			(show_name no)
@@
 			(project "CyberwatchV1B"
 				(path "/68fdecbc-307b-4175-ba1b-687d291eebec/ea0244fb-2f59-483a-a25c-2656c752d645"
-					(reference "SW1")
+					(reference "SW2")
 					(unit 1)
 				)
@@
 		(dnp no)
 		(fields_autoplaced yes)
-		(property "Reference" "#PWR022"
+		(property "Reference" "#PWR028"
 			(at 149.86 93.98 0)
 			(hide yes)
@@
 			(project "CyberwatchV1B"
 				(path "/68fdecbc-307b-4175-ba1b-687d291eebec/ea0244fb-2f59-483a-a25c-2656c752d645"
-					(reference "#PWR022")
+					(reference "#PWR028")
 					(unit 1)
 				)
@@
 		(in_pos_files yes)
 		(dnp no)
-		(property "Reference" "SW2"
+		(property "Reference" "SW3"
 			(at 164.338 108.966 0)
 			(show_name no)
@@
 			(project "CyberwatchV1B"
 				(path "/68fdecbc-307b-4175-ba1b-687d291eebec/ea0244fb-2f59-483a-a25c-2656c752d645"
-					(reference "SW2")
+					(reference "SW3")
 					(unit 1)
 				)
@@
 		(in_pos_files yes)
 		(dnp no)
-		(property "Reference" "#PWR044"
+		(property "Reference" "#PWR029"
 			(at 204.47 96.52 0)
 			(hide yes)
@@
 			(project "CyberwatchV1B"
 				(path "/68fdecbc-307b-4175-ba1b-687d291eebec/ea0244fb-2f59-483a-a25c-2656c752d645"
-					(reference "#PWR044")
-					(unit 1)
-				)
+					(reference "#PWR029")
+					(unit 1)
+				)

Commit message: PCB design finalisation
Parts:
- J6: MPN (none) -> SM03B-SRSS-TB(LF)(SN)
- SW2, SW3: MPN (none) -> KMR231NG LFS
Changed lines of the file:
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@@
+			)
+		)
+		(property "MPN" " SM03B-SRSS-TB(LF)(SN)"
+			(at 195.58 99.06 0)
+			(hide yes)
+			(show_name no)
+			(do_not_autoplace no)
+			(effects
+				(font
+					(size 1.27 1.27)
+				)
 			)
 		)
@@
 			)
 		)
+		(property "MPN" " KMR231NG LFS"
+			(at 163.83 93.98 0)
+			(hide yes)
+			(show_name no)
+			(do_not_autoplace no)
+			(effects
+				(font
+					(size 1.27 1.27)
+				)
+			)
+		)
 		(pin "2"
 		)
@@
 			(at 163.83 104.14 0)
 			(hide yes)
+			(show_name no)
+			(do_not_autoplace no)
+			(effects
+				(font
+					(size 1.27 1.27)
+				)
+			)
+		)
+		(property "MPN" " KMR231NG LFS"
+			(at 163.83 104.14 0)
+			(hide yes)
