File: design/electronics2/CyberwatchV1B/input_right.kicad_sch (KiCad schematic)
At the start: 0 parts

Commit message: electronics progres
Parts:
- added J8: Conn_01x07_main, symbol Connector_Generic:Conn_01x07
- added SW4: SW_Push, Button_Switch_SMD:SW_Push_1P1T_NO_CK_KMR2, symbol Switch:SW_Push
- added U5: MT6701CT, Package_SO:SO-8_3.9x4.9mm_P1.27mm, symbol Sensor_Magnetic:MT6701CT
Connections:
- new net +3.3V: U5.1 (VDD)
- new net BTN_3: U5.5 (PUSH)
- new net BTN_4: SW4.2
- new net GND: SW4.1, U5.2 (MODE), U5.4 (GND)
- new net SCL: U5.7 (B)
- new net SDA: U5.6 (A)
- no-connect marks 0 -> 2

Commit message: schematic complete
Parts:
- J8: value Conn_01x07_main -> Conn_01x07_input_right
Connections:
- net +3.3V: now also J8.2 (Pin_2)
- net BTN_3: now also J8.5 (Pin_5)
- net BTN_4: now also J8.6 (Pin_6)
- net GND: now also J8.1 (Pin_1), J8.7 (Pin_7)
- net SCL: now also J8.4 (Pin_4)
- net SDA: now also J8.3 (Pin_3)

Commit message: sync
Parts:
- J8: value Conn_01x07_input_right -> Conn_01x07_IR_main; footprint (none) -> Connector_JST:JST_SH_SM07B-SRSS-TB_1x07-1MP_P1.00mm_Horizontal
Changed lines of the file:
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@@
 			)
 		)
-		(property "Value" "Conn_01x07_input_right"
+		(property "Value" "Conn_01x07_IR_main"
 			(at 80.01 44.958 0)
 			(show_name no)
@@
 			)
 		)
-		(property "Footprint" ""
+		(property "Footprint" "Connector_JST:JST_SH_SM07B-SRSS-TB_1x07-1MP_P1.00mm_Horizontal"
 			(at 80.01 58.42 0)
 			(hide yes)

Commit message: pcb design
Parts:
- added C4: 100nF, Capacitor_SMD:C_0603_1608Metric, symbol Device:C_Small
- J7: renamed from J8; KiLib_Generator (none) -> connector/SMD_single_row_plus_mounting_pad
- U5: KiLib_Generator (none) -> package/gullwing
Connections:
- net +3.3V: now also C4.1; no longer U5.1 (VDD)
- new net: C4.2, U5.1 (VDD)

Commit message: PCB design finalisation
Parts:
- C4: MPN (none) -> CL10B104KB8NNNC
- J7: MPN (none) -> SM07B-SRSS-TB(LF)(SN)
- SW4: MPN (none) -> KMR231NG LFS
- U5: MPN (none) -> MT6701CT-STD
Changed lines of the file:
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@@
+			)
+		)
+		(property "MPN" "MT6701CT-STD"
+			(at 134.62 66.04 0)
+			(hide yes)
+			(show_name no)
+			(do_not_autoplace no)
+			(effects
+				(font
+					(size 1.27 1.27)
+				)
 			)
 		)
@@
 			)
 		)
+		(property "MPN" " SM07B-SRSS-TB(LF)(SN)"
+			(at 80.01 58.42 0)
+			(hide yes)
+			(show_name no)
+			(do_not_autoplace no)
+			(effects
+				(font
+					(size 1.27 1.27)
+				)
+			)
+		)
 		(pin "2"
 		)
@@
 			)
 		)
+		(property "MPN" "CL10B104KB8NNNC"
+			(at 134.62 39.37 0)
+			(hide yes)
+			(show_name no)
+			(do_not_autoplace no)
+			(effects
+				(font
+					(size 1.27 1.27)
+				)
+			)
+		)
 		(pin "1"
 		)
@@
 			(at 134.62 101.6 0)
 			(hide yes)
+			(show_name no)
+			(do_not_autoplace no)
+			(effects
+				(font
+					(size 1.27 1.27)
+				)
+			)
+		)
+		(property "MPN" " KMR231NG LFS"
+			(at 134.62 101.6 0)
+			(hide yes)
