File: design/electronics2/CyberwatchV1B/main.kicad_sch (KiCad schematic)
At the start: 6 parts, among them J1 Micro_SD_Card, J2 Conn_01x08_Display, U1 XIAO-ESP32-S3-Plus-SMD, U2 MCP23017x-x-ML, U3 DS3231MZ

Commit message: power schematic finalisation
Other:
- moved on the sheet: J2, U2
Changed lines of the file:
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@@
 	(paper "A4")
 	(no_connect
-		(at 72.39 99.06)
+		(at 80.01 92.71)
 	)
 	(no_connect
@@
 	)
 	(no_connect
-		(at 67.31 99.06)
+		(at 74.93 92.71)
 	)
 	(no_connect
-		(at 54.61 99.06)
+		(at 62.23 92.71)
 	)
 	(no_connect
-		(at 59.69 99.06)
+		(at 67.31 92.71)
 	)
 	(no_connect
-		(at 74.93 99.06)
+		(at 82.55 92.71)
 	)
 	(no_connect
-		(at 62.23 99.06)
+		(at 69.85 92.71)
 	)
 	(no_connect
-		(at 57.15 99.06)
+		(at 64.77 92.71)
 	)
 	(no_connect
-		(at 52.07 99.06)
+		(at 59.69 92.71)
 	)
 	(no_connect
-		(at 49.53 99.06)
+		(at 57.15 92.71)
 	)
 	(no_connect
-		(at 64.77 99.06)
+		(at 72.39 92.71)
 	)
 	(no_connect
@@
 	(wire
 		(pts
-			(xy 92.71 27.94) (xy 102.87 27.94)
+			(xy 74.93 53.34) (xy 85.09 53.34)
 		)
 		(stroke
@@
 	(wire
 		(pts
-			(xy 92.71 38.1) (xy 104.14 38.1)
+			(xy 74.93 63.5) (xy 86.36 63.5)
 		)
 		(stroke
@@
 	(wire
 		(pts
-			(xy 92.71 30.48) (xy 102.87 30.48)
+			(xy 74.93 55.88) (xy 85.09 55.88)
 		)
 		(stroke
@@
 	(wire
 		(pts
-			(xy 92.71 45.72) (xy 96.52 45.72)
+			(xy 74.93 71.12) (xy 78.74 71.12)
 		)
 		(stroke
@@
 	(wire
 		(pts
-			(xy 92.71 40.64) (xy 101.6 40.64)
+			(xy 74.93 66.04) (xy 83.82 66.04)
 		)
 		(stroke
@@
 	(wire
 		(pts
-			(xy 99.06 43.18) (xy 92.71 43.18)
+			(xy 81.28 68.58) (xy 74.93 68.58)
 		)
 		(stroke
@@
 	)
 	(label "SPI_CLK"
-		(at 92.71 35.56 0)
+		(at 74.93 60.96 0)
 		(effects
 			(font
@@
 	)
 	(label "I2C_SCL"
-		(at 90.17 124.46 270)
+		(at 97.79 118.11 270)
 		(effects
 			(font
@@
 	)
 	(label "SPI_MOSI"
-		(at 92.71 33.02 0)
+		(at 74.93 58.42 0)
 		(effects
 			(font
@@
 	)
 	(label "I2C_SDA"
-		(at 87.63 124.46 270)
+		(at 95.25 118.11 270)
 		(effects
 			(font
@@
 		)
 	)
+	(hierarchical_label "VBAT_RAW"
+		(shape input)
+		(at 101.6 19.05 270)
+		(effects
+			(font
+				(size 1.27 1.27)
+			)
+			(justify right)
+		)
+	)
+	(hierarchical_label "VBAT_SWITCHED"
+		(shape input)
+		(at 88.9 19.05 270)
+		(effects
+			(font
+				(size 1.27 1.27)
+			)
+			(justify right)
+		)
+	)
+	(hierarchical_label "BTN_2"
+		(shape input)
+		(at 25.4 88.9 0)
+		(effects
+			(font
+				(size 1.27 1.27)
+			)
+			(justify left)
+		)
+	)
+	(hierarchical_label "BTN_1"
+		(shape input)
+		(at 25.4 63.5 0)
+		(effects
+			(font
+				(size 1.27 1.27)
+			)
+			(justify left)
+		)
+	)
+	(hierarchical_label "GND"
+		(shape input)
+		(at 114.3 19.05 270)
+		(effects
+			(font
+				(size 1.27 1.27)
+			)
+			(justify right)
+		)
+	)
 	(symbol
 		(lib_id "power:GND")
-		(at 102.87 30.48 90)
+		(at 85.09 55.88 90)
 		(unit 1)
 		(body_style 1)
@@
 		(fields_autoplaced yes)
 		(property "Reference" "#PWR01"
-			(at 109.22 30.48 0)
+			(at 91.44 55.88 0)
 			(hide yes)
 			(show_name no)
@@
 		)
 		(property "Value" "GND"
-			(at 106.68 30.4799 90)
+			(at 88.9 55.8799 90)
 			(show_name no)
 			(do_not_autoplace no)
@@
 		)
 		(property "Footprint" ""
-			(at 102.87 30.48 0)
+			(at 85.09 55.88 0)
 			(hide yes)
 			(show_name no)
@@
 		)
 		(property "Datasheet" ""
-			(at 102.87 30.48 0)
+			(at 85.09 55.88 0)
 			(hide yes)
 			(show_name no)
@@
 		)
 		(property "Description" "Power symbol creates a global label with name \"GND\" , ground"
-			(at 102.87 30.48 0)
+			(at 85.09 55.88 0)
 			(hide yes)
 			(show_name no)
@@
 	(symbol
 		(lib_id "Interface_Expansion:MCP23017x-x-ML")
-		(at 69.85 111.76 270)
+		(at 77.47 105.41 270)
 		(mirror x)
 		(unit 1)
@@
 		(dnp no)
 		(property "Reference" "U2"
-			(at 82.042 112.014 90)
+			(at 89.662 105.664 90)
 			(show_name no)
 			(do_not_autoplace no)
@@
 		)
 		(property "Value" "MCP23017x-x-ML"
-			(at 68.326 111.76 90)
+			(at 75.946 105.41 90)
 			(show_name no)
 			(do_not_autoplace no)
@@
 		)
 		(property "Footprint" "Package_DFN_QFN:QFN-28-1EP_6x6mm_P0.65mm_EP4.25x4.25mm"
-			(at 44.45 106.68 0)
+			(at 52.07 100.33 0)
 			(hide yes)
 			(show_name no)
@@
 		)
 		(property "Datasheet" "https://ww1.microchip.com/downloads/aemDocuments/documents/APID/ProductDocuments/DataSheets/MCP23017-Data-Sheet-DS20001952.pdf"
-			(at 41.91 106.68 0)
+			(at 49.53 100.33 0)
 			(hide yes)
 			(show_name no)
@@
 		)
 		(property "Description" "16-bit I/O expander, I2C, interrupts, w pull-ups, GPA7/GPB7 output only (https://microchip.my.site.com/s/article/GPA7---GPB7-Cannot-Be-Used-as-Inputs-In-MCP23017), QFN-28"
-			(at 69.85 111.76 0)
+			(at 77.47 105.41 0)
 			(hide yes)
 			(show_name no)
@@
 	(symbol
 		(lib_id "power:+3.3V")
-		(at 102.87 27.94 270)
+		(at 85.09 53.34 270)
 		(unit 1)
 		(body_style 1)
@@
 		(fields_autoplaced yes)
 		(property "Reference" "#PWR05"
-			(at 99.06 27.94 0)
+			(at 81.28 53.34 0)
 			(hide yes)
 			(show_name no)
@@
 		)
 		(property "Value" "+3.3V"
-			(at 106.68 27.9399 90)
+			(at 88.9 53.3399 90)
 			(show_name no)
 			(do_not_autoplace no)
@@
 		)
 		(property "Footprint" ""
-			(at 102.87 27.94 0)
+			(at 85.09 53.34 0)
 			(hide yes)
 			(show_name no)
@@
 		)
 		(property "Datasheet" ""
-			(at 102.87 27.94 0)
+			(at 85.09 53.34 0)
 			(hide yes)
 			(show_name no)
@@
 		)
 		(property "Description" "Power symbol creates a global label with name \"+3.3V\""
-			(at 102.87 27.94 0)
+			(at 85.09 53.34 0)
 			(hide yes)
 			(show_name no)
@@
 	(symbol
 		(lib_id "CY_library:Conn_01x08")
-		(at 87.63 35.56 0)
+		(at 69.85 60.96 0)
 		(mirror y)
 		(unit 1)
@@
 		(dnp no)
 		(property "Reference" "J2"
-			(at 82.804 35.56 0)
+			(at 65.024 60.96 0)
 			(show_name no)
 			(do_not_autoplace no)
@@
 		)
 		(property "Value" "Conn_01x08_Display"
-			(at 94.742 24.13 0)
+			(at 76.962 49.53 0)
 			(show_name no)
 			(do_not_autoplace no)
@@
 		)
 		(property "Footprint" ""
-			(at 87.63 35.56 0)
+			(at 69.85 60.96 0)
 			(hide yes)
 			(show_name no)
@@
 		)
 		(property "Datasheet" ""
-			(at 87.63 35.56 0)
+			(at 69.85 60.96 0)
 			(hide yes)
 			(show_name no)
@@
 		)
 		(property "Description" "Display connector, single row, 01x08, script generated (kicad-library-utils/schlib/autogen/connector/)"
-			(at 83.058 21.59 0)
-			(hide yes)
-			(show_name no)
+			(at 65.278 46.99 0)
+			(hide yes)
+			(show_name no)

Commit message: documentation and electronics main board progress
Parts:
- added R3, R4, R5, R6, R7: 10k, symbol Device:R
Connections:
- net I2C_SCL is gone; now on net SCL: U1.6 (D5), U2.8 (SCL)
- net I2C_SDA is gone; now on net SDA: U1.5 (D4), U2.9 (SDA)
- net BTN_1: now also U2.19 (GPA2)
- net BTN_2: now also U2.20 (GPA3)
- net GND: now also U1.13 (GND)
- net VBAT_SWITCHED: now also U1.32 (VBAT)
- net at U2.17 (GPA0): now also J2.7 (Pin_7)
- net at U2.18 (GPA1): now also J2.8 (Pin_8)
- net BTN_3: now reaches U2.21 (GPA4)
- net BTN_4: now reaches U2.22 (GPA5)
- net ALRT: now reaches U2.25 (GPB0)
- net at U1.10 (D9): now also J1.2 (DAT3/CD)
- net at U1.2 (D1): now also J2.5 (CS)
- net at U1.4 (D3): now also J2.6 (Pin_6)
- net SPI_MISO: now reaches U1.8 (D7)
- net SPI_MISO: now also J1.7 (DAT0)
- net SDA: now reaches U3.7 (SDA)
- net SCL: now reaches U3.8 (SCL)
- no-connect marks 12 -> 27
Other:
- moved on the sheet: BT1, J1, J2, U1, U2, U3

Commit message: electronics progres
Parts:
- added C1, C2: 100nF, Capacitor_SMD:C_0603_1608Metric, symbol Device:C_Small
- added J4: Conn_01x07_power, symbol Connector_Generic:Conn_01x07
- added J5: Conn_01x03_input_left, symbol Connector_Generic:Conn_01x03
- added J6: Conn_01x07_input_right, symbol Connector_Generic:Conn_01x07
- added R10: 10k, Resistor_SMD:R_0603_1608Metric, symbol Device:R
- added R8, R9: 4.7k, Resistor_SMD:R_0603_1608Metric, symbol Device:R
- BT1: footprint (none) -> Battery:BatteryHolder_Keystone_3000_1x12mm
- J1: footprint (none) -> Connector_Card:microSD_HC_Molex_47219-2001
- J2: footprint (none) -> Connector_JST:JST_GH_SM08B-GHS-TB_1x08-1MP_P1.25mm_Horizontal
- R3, R4, R5, R6, R7: footprint (none) -> Resistor_SMD:R_0603_1608Metric
Connections:
- net +3.3V: now also R6.1, R7.1, U1.12 (3V3_OUT), U2.14 (~{RESET}), C1.1, R10.1; no longer U3.2 (VCC)
- net GND: now also BT1.2 (-), J1.SH (SHIELD), U1.27 (GND), U1.34 (PAD), U2.11 (A0), U2.12 (A1), U2.13 (A2), U2.29 (EP), U2.6 (V_{SS})
- net SCL: now also R9.1; no longer U1.6 (D5)
- net SDA: now also R8.1; no longer U1.5 (D4)
- net SPI_MISO: now also R5.1; no longer J1.7 (DAT0)
- net SPI_MOSI: now also R4.1; no longer J1.3 (CMD)
- net VBAT_RAW: now also C2.2
- net at U2.5 (V_{DD}): now also C1.2
- net at U1.10 (D9): now also R3.1; no longer J1.2 (DAT3/CD)
- net at R3.2: now also J1.2 (DAT3/CD)
- net at U3.4 (~{RST}): now also R10.2
- net at R4.2: now also J1.3 (CMD)
- net at J1.1 (DAT2): now also R7.2
- net at J1.8 (DAT1): now also R6.2
- net at R5.2: now also J1.7 (DAT0)
- new net: C2.1, U3.2 (VCC)
- new net: R8.2, U1.5 (D4)
- new net: R9.2, U1.6 (D5)
- no-connect marks 27 -> 33
Other:
- moved on the sheet: BT1, J1, R3, R4, R6, R7, U1, U2, U3

Commit message: schematic complete
Parts:
- removed J4: Conn_01x07_power, symbol Connector_Generic:Conn_01x07
- added J10: Conn_01x07_power, symbol Connector_Generic:Conn_01x07
Connections:
- net +3.3V: now also J6.2 (Pin_2)
- net BTN_1: now also J5.2 (Pin_2)
- net BTN_2: now also J5.3 (Pin_3)
- net BTN_3: now also J6.5 (Pin_5)
- net BTN_4: now also J6.6 (Pin_6)
- net GND: now also J5.1 (Pin_1), J6.1 (Pin_1), J6.7 (Pin_7), J10.3 (Pin_3), J10.7 (Pin_7)
- net SCL: now also J6.4 (Pin_4), J10.5 (Pin_5)
- net SDA: now also J6.3 (Pin_3), J10.4 (Pin_4)
- net VBAT_RAW: now also J10.1 (Pin_1)
- net VBAT_SWITCHED: now also J10.2 (Pin_2)
- net ALRT renamed PWR_ALRT
- net PWR_ALRT: now also J10.6 (Pin_6)
Other:
- moved on the sheet: J5, J6

Commit message: sync
Parts:
- J10: value Conn_01x07_power -> Conn_01x07_M_power; footprint (none) -> Connector_JST:JST_SH_SM07B-SRSS-TB_1x07-1MP_P1.00mm_Horizontal
- J5: value Conn_01x03_input_left -> Conn_01x03_M_input_left; footprint (none) -> Connector_JST:JST_SH_SM03B-SRSS-TB_1x03-1MP_P1.00mm_Horizontal
- J6: value Conn_01x07_input_right -> Conn_01x07_M_input_right; footprint (none) -> Connector_JST:JST_SH_SM07B-SRSS-TB_1x07-1MP_P1.00mm_Horizontal
Changed lines of the file:
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@@
 			)
 		)
-		(property "Value" "Conn_01x07_input_right"
+		(property "Value" "Conn_01x07_M_input_right"
 			(at 261.62 61.468 0)
 			(show_name no)
@@
 			)
 		)
-		(property "Footprint" ""
+		(property "Footprint" "Connector_JST:JST_SH_SM07B-SRSS-TB_1x07-1MP_P1.00mm_Horizontal"
 			(at 261.62 74.93 0)
 			(hide yes)
@@
 		(dnp no)
 		(property "Reference" "U3"
-			(at 165.862 65.532 0)
+			(at 165.862 66.294 0)
 			(show_name no)
 			(do_not_autoplace no)
@@
 		)
 		(property "Value" "DS3231MZ"
-			(at 165.862 63.5 0)
+			(at 165.862 64.262 0)
 			(show_name no)
 			(do_not_autoplace no)
@@
 			)
 		)
-		(property "Value" "Conn_01x03_input_left"
+		(property "Value" "Conn_01x03_M_input_left"
 			(at 52.578 61.468 0)
 			(show_name no)
@@
 			)
 		)
-		(property "Footprint" ""
+		(property "Footprint" "Connector_JST:JST_SH_SM03B-SRSS-TB_1x03-1MP_P1.00mm_Horizontal"
 			(at 54.61 69.85 0)
 			(hide yes)
@@
 			)
 		)
-		(property "Value" "Conn_01x07_power"
+		(property "Value" "Conn_01x07_M_power"
 			(at 115.824 21.59 0)
 			(show_name no)
@@
 			)
 		)
-		(property "Footprint" ""
+		(property "Footprint" "Connector_JST:JST_SH_SM07B-SRSS-TB_1x07-1MP_P1.00mm_Horizontal"
 			(at 104.14 33.02 0)
 			(hide yes)

Commit message: pcb design
Parts:
- removed J10: Conn_01x07_M_power, Connector_JST:JST_SH_SM07B-SRSS-TB_1x07-1MP_P1.00mm_Horizontal, symbol Connector_Generic:Conn_01x07
- added C2: 100nF, Capacitor_SMD:C_0603_1608Metric, symbol Device:C_Small
- added J1: Conn_01x02_M_Battery, Connector_JST:JST_PH_S2B-PH-SM4-TB_1x02-1MP_P2.00mm_Horizontal, symbol Connector:Conn_01x02_Socket
- added Q1: AO3401A, Package_TO_SOT_SMD:SOT-23, symbol Transistor_FET:AO3401A
- added R1: 100k, Resistor_SMD:R_0603_1608Metric, symbol Device:R
- added R2: 33, Resistor_SMD:R_0603_1608Metric, symbol Device:R
- added SW1: SW_power, Button_Switch_SMD:SW_DIP_SPSTx01_Slide_Copal_CHS-01A_W5.08mm_P1.27mm_JPin, symbol Switch:SW_SPST
- added U1: MAX17048, Package_DFN_QFN:TDFN-8-1EP_2x2mm_P0.5mm_EP0.8x1.2mm, symbol CY_library:MAX17048
- C1: renamed from C2; KiLib_Generator (none) -> SMD_2terminal_chip_molded
- C3: renamed from C1; KiLib_Generator (none) -> SMD_2terminal_chip_molded
- J2: renamed from J5; KiLib_Generator (none) -> connector/SMD_single_row_plus_mounting_pad
- J3: renamed from J6; KiLib_Generator (none) -> connector/SMD_single_row_plus_mounting_pad
- J4: renamed from J2; value Conn_01x08_Display -> Conn_01x08_M_Display; KiLib_Generator (none) -> connector/SMD_single_row_plus_mounting_pad
- R10: renamed from R9; KiLib_Generator (none) -> SMD_2terminal_chip_molded
- R3: renamed from R10; KiLib_Generator (none) -> SMD_2terminal_chip_molded
- R4: renamed from R7; KiLib_Generator (none) -> SMD_2terminal_chip_molded
- R5: renamed from R3; KiLib_Generator (none) -> SMD_2terminal_chip_molded
- R6: renamed from R4; KiLib_Generator (none) -> SMD_2terminal_chip_molded
- R7: renamed from R5; KiLib_Generator (none) -> SMD_2terminal_chip_molded
- R8: renamed from R6; KiLib_Generator (none) -> SMD_2terminal_chip_molded
- R9: renamed from R8; KiLib_Generator (none) -> SMD_2terminal_chip_molded
- U2: renamed from U3; KiLib_Generator (none) -> package/gullwing
- U4: renamed from U2; KiLib_Generator (none) -> package/no_lead
- renumbered J1 to J5, U1 to U3
Connections:
- net GND: now also C2.1, J1.2 (Pin_2), SW1.2 (B), U1.3 (CTG), U1.4 (GND), U1.8 (QSTRT)
- net PWR_ALRT: now also U1.5 (ALRT)
- net SCL: now also U1.7 (SCL)
- net SDA: now also U1.6 (SDA)
- net VBAT_RAW renamed S
- net S: now also C2.2, J1.1 (Pin_1), Q1.2 (S), R1.1, U1.1 (VDD)
- net VBAT_SWITCHED renamed D
- net D: now also Q1.3 (D)
- new net: R2.1, SW1.1 (A)
- new net G: Q1.1 (G), R1.2, R2.2
Other:
- moved on the sheet: BT1, C1, C3, J2, J3, J4, J5, R10, R3, R4, R5, R6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

Commit message: PCB design finalisation
Parts:
- BT1: MPN (none) -> Keystone 3000
- C1, C2, C3: MPN (none) -> CL10B104KB8NNNC
- J1: MPN (none) -> S2B-PH-SM4-TB(LF)(SN)
- J2: MPN (none) -> SM03B-SRSS-TB(LF)(SN)
- J3: MPN (none) -> SM07B-SRSS-TB(LF)(SN)
- J4: MPN (none) -> SM08B-GHS-TB(LF)(SN)
- J5: MPN (none) -> 47219-2001
- Q1: MPN (none) -> AO3401A
- R1: MPN (none) -> RC0603FR-07100KL
- R10, R9: MPN (none) -> RC0603FR-074K7L
- R2: MPN (none) -> RC0603FR-0733RL
- R3, R4, R5, R6, R7, R8: MPN (none) -> RC0603FR-0710KL
- SW1: MPN (none) -> CHS-01A
- U1: MPN (none) -> MAX17048G+T10
- U2: MPN (none) -> DS3231MZ+
- U4: MPN (none) -> MCP23017-E/ML
